File: PCB/devboard/devboard.kicad_pcb (KiCad board)
At the start: 2 copper layers, 27 x 43.4 mm, 45 parts, among them J1 Conn_01x13_Pin, J3 Micro_SD_Card, J4 USB_C_Receptacle_USB2.0_14P, SW1 SW_Push, SW2 SW_Push, U1 ESP32-C6, U2 TPS62172DSG, U3 W25Q64JVSSIQ, Y1 C521661, Y3 Crystal

Commit message: silkscreeeen
Parts:
- added G***: LOGO, LOGO, F.Cu at (15.6, 18.1)
- added G***: LOGO, LOGO, B.Cu at (16.4, 15.6)
- added G***: LOGO, LOGO, B.Cu at (5.90, 15.7)
- L1: value 2uH -> 2.2uH
- moved JP1 0.75 mm to (22.0, 43.6)
Connections:
- J1 pad 6: /GPIO10 -> /GPIO11
- J1 pad 7: /GPIO11 -> /GPIO10
Routing:
- net /GPIO11: track 19.6 -> 15.0 mm
- net Net-(JP1-A): track 1.68 -> 3.82 mm
- net /GPIO10: track 13.8 -> 14.8 mm
- net +3.3V: track 156.4 -> 155.8 mm
Other:
- board text added: "1"
- board text added: "10"
- board text added: "10 GPIOs"
- board text added: "2"
- board text added: "2.4GHz"
- board text added: "3"
- board text added: "3.3v"
- board text added: "32kHz"
- board text added: "4"
- board text added: "40MHz"
- board text added: "5"
- board text added: "5v"
- board text added: "6"
- board text added: "64Mbit"
- board text added: "7"
- board text added: "8"
- board text added: "9"
- board text added: "<256GB"
- board text added: "BIG CAPS"
- board text added: "BOOT"
- board text added: "C6dev"
- board text added: "ESP32-C6"
- board text added: "GND"
- board text added: "GPIO11"
- board text added: "GPIO16"
- board text added: "GPIO17"
- board text added: "GPIO2"
- board text added: "GPIO3"
- board text added: "GPIO4"
- board text added: "GPIO5"
- board text added: "GPIO6"
- board text added: "GPIO7"
- board text added: "RESET"
- board text added: "USB 2.0"
- board text added: "cut = no power LED"
- board text added: "github.com/ImShyMike/C6dev"
- board text added: "the sad RF corner"

Commit message: finishing up
Parts:
- removed the G*** at (15.6, 18.1)
- added G***: LOGO, LOGO, F.Cu at (14.2, 18.1)
- added G***: LOGO, LOGO, F.Cu at (16.7, 18.1)
- added G***: LOGO, LOGO, B.Cu at (33.1, 22.1)
- added G***: LOGO, LOGO, B.Cu at (34.6, 45.8)
- added G***: LOGO, LOGO, B.Cu at (34.1, 39.0)
- added G***: LOGO, LOGO, B.Cu at (34.4, 29.4)
- moved JP1 0.75 mm to (21.2, 43.6)
- moved G*** 0.30 mm to (5.60, 15.7)
Connections:
- J1 pad 4: /GPIO16 -> /GPIO17
- J1 pad 5: /GPIO17 -> /GPIO16
Routing:
- net /GPIO16: track 30.5 -> 23.6 mm
- net /GPIO17: track 23.1 -> 27.2 mm
- net Net-(JP1-A): track 3.82 -> 1.11 mm
- net GND: track 26.8 -> 25.8 mm
Other:
- board text added: "GPIO10"
- board text added: "GPIO2/FSPIQ/ADC"
- board text added: "GPIO3/ADC"
- board text added: "MTCK/GPIO6/FSPICLI/ADC"
- board text added: "MTDI/GPIO5/FSPIWP/ADC"
- board text added: "MTDO/GPIO7/FSPID"
- board text added: "MTMS/GPIO4/FSPIHD/ADC"
- board text added: "RX/GPIO17/FSPICS1"
- board text added: "TX/GPIO16/FSPICS0"
- board text removed: "GPIO16"
- board text removed: "GPIO17"
- board text removed: "GPIO2"
- board text removed: "GPIO3"
- board text removed: "GPIO4"
- board text removed: "GPIO5"
- board text removed: "GPIO6"
- board text removed: "GPIO7"
