File: PCB/devboard/devboard.kicad_sch (KiCad schematic)
At the start: 0 parts

Commit message: update
Parts:
- added AE1: Antenna_Shield, Connector_Coaxial:U.FL_Hirose_U.FL-R-SMT-1_Vertical, symbol Device:Antenna_Shield
- added C1: 100nF, symbol Device:C
- added C2, C3: 12pF, symbol Device:C_Small
- added C4, C5: 6.8pF, symbol Device:C_Small
- added C6: 10uF, symbol Device:C_Small
- added C7: 22uF, symbol Device:C_Small
- added D1: LED, symbol Device:LED
- added J1, J2: Conn_01x20_Socket, symbol Connector:Conn_01x20_Socket
- added J3: Micro_SD_Card, symbol Connector:Micro_SD_Card
- added J4: USB_C_Receptacle_USB2.0_14P, symbol Connector:USB_C_Receptacle_USB2.0_14P
- added L1: 2uH, symbol Device:L_Small
- added R1, R4: 10k, symbol Device:R
- added R10, R11, R12, R2, R3, R8, R9: 10k, symbol Device:R_Small
- added R5, R6: 5.1kΩ, symbol Device:R
- added R7: 100k, symbol Device:R_Small
- added SW1, SW2: SW_Push, symbol Switch:SW_Push
- added U1: ESP32-C6, Package_DFN_QFN:QFN-40-1EP_5x5mm_P0.4mm_EP3.6x3.6mm, symbol EXPRESSIF:ESP32-C6
- added U2: TPS62172DSG, Package_SON:WSON-8-1EP_2x2mm_P0.5mm_EP0.9x1.6mm_ThermalVias, symbol Regulator_Switching:TPS62172DSG
- added U3: W25Q64JVSSIQ, W25Q64JVSSIQ:SOIC-8_5P28X5P28_WIN, symbol W25Q64JVSSIQ:W25Q64JVSSIQ
- added Y1: C521661, symbol Device:Crystal_GND24
- added Y2: C252396, symbol Device:Crystal_GND24
Connections:
- new net: J4.A5 (CC1), R6.2
- new net: L1.1, U2.7 (SW)
- new net: R7.2, U2.8 (PG)
- new net: J4.B5 (CC2), R5.2
- new net +3.3V: C7.1, J3.4 (VDD), L1.2, R1.1, R10.2, R11.2, R12.2, R2.1, R3.2, R4.1, R7.1, R8.1, R9.2, U1.2 (VDDA3P3), U1.28 (VDDPST2), U1.3 (VDDA3P3), U1.37 (VDDA1), U1.40 (VDDA2), U1.5 (VDDPST1), U2.6 (VOS)
- new net +5V: C6.2, J4.A4 (VBUS), J4.A9 (VBUS), J4.B4 (VBUS), J4.B9 (VBUS), U2.2 (VIN), U2.3 (EN)
- new net ANT: AE1.1 (A), U1.1 (ANT)
- new net BOOT: R8.2, U1.14 (GPIO8)
- new net BOOT_BTN: R1.2, SW1.1, U1.15 (GPIO9)
- new net GND: AE1.2 (Shield), C1.2, C2.1, C3.2, C4.1, C5.2, C6.1, C7.2, J3.6 (VSS), J3.9 (SHIELD), J4.A1 (GND), J4.A12 (GND), J4.B1 (GND), J4.B12 (GND), J4.S1 (SHIELD), R5.1, R6.1, SW1.2, SW2.2, U1.41 (GND), U2.1 (PGND), U2.4 (AGND), U2.5 (FB), U2.9 (PAD), U3.4 (GND), Y1.2, Y1.4, Y2.2, Y2.4
- new net RESET_BTN: C1.1, R4.2, SW2.1, U1.4 (CHIP_PU)
- new net SD_CLK: J3.5 (CLK), U1.32 (GPIO19/SDIO_CLK/FSPICS3)
- new net SD_CMD: J3.3 (CMD), R12.1, U1.31 (GPIO18/SDIO_CMD/FSPICS2)
- new net SD_DATA0: J3.7 (DAT0), R9.1, U1.33 (GPIO20/SDIO_DATA0/FSPICS4)
- new net SD_DATA1: J3.8 (DAT1), R3.1, U1.34 (GPIO21/SDIO_DATA1/FSPICS5)
- new net SD_DATA2: J3.1 (DAT2), R10.1, U1.35 (GPIO22/SDIO_DATA2)
- new net SD_DATA3: J3.2 (DAT3/CD), R11.1, U1.36 (GPIO23/SDIO_DATA3)
- new net SPICLK: U1.25 (SPICLK/GPIO29), U3.6 (CLK)
- new net SPICS0: U1.20 (SPICS0/GPIO24), U3.1 (/CS)
- new net SPID: U1.26 (SPID/GPIO30), U3.5 (DI(IO0))
- new net SPIHD: U1.24 (SPIHD/GPIO28), U3.7 (/HOLD_OR_/RESET(IO3))
- new net SPIQ: U1.21 (SPIQ/GPIO25), U3.2 (DO(IO1))
- new net SPIWP: U1.22 (SPIWP/GPIO26), U3.3 (/WP(IO2))
- new net USB_D+: J4.A6 (D+), J4.B6 (D+), U1.19 (GPIO13/USB_D+)
- new net USB_D-: J4.A7 (D-), J4.B7 (D-), U1.18 (GPIO12/USB_D-)
- new net USB_JTAG: R2.2, U1.27 (GPIO15)
- new net VDD_SPI: U1.23 (VDD_SPI/GPIO27), U3.8 (VCC)
- new net XTAL_32k_N: C5.1, U1.7 (GPIO1/XTAL_32K_N/ADC1_CH1), Y2.1
- new net XTAL_32k_P: C4.2, U1.6 (GPIO0/XTAL_32K_P/ADC1_CH0), Y2.3
- new net XTAL_N: C2.2, U1.38 (XTAL_N), Y1.3
- new net XTAL_P: C3.1, U1.39 (XTAL_P), Y1.1
Other:
- note added: "32Khz Crystal Oscillator"
- note added: "40MHz Crystal Oscillator"
- note added: "Boot Button"
- note added: "Buttons"
- note added: "Crystals"
- note added: "MicroSD Card"
- note added: "Quad SPI 64Mbit Flash"
- note added: "Reset Button"
- note added: "SDIO Pull-ups"
- note added: "Step-Down Converter"
- note added: "USB C 2.0"

Commit message: finished schematic
Parts:
- removed J1, J2: Conn_01x20_Socket, symbol Connector:Conn_01x20_Socket
- added C10, C11, C12, C15, C8, C9: 100nF, symbol Device:C_Small
- added C13: 470uF, symbol Device:C_Small
- added C14: 100uF, symbol Device:C_Small
- added C16: 100nF, symbol Device:C
- added J1: Conn_01x10_Pin, symbol Connector:Conn_01x10_Pin
- added R13: 10k, symbol Device:R_Small
Connections:
- net +3.3V: now also C10.1, C11.1, C12.1, C13.1, C14.1, C8.1, C9.1, R13.2
- net BOOT_BTN: now also C16.1
- net GND: now also D1.1 (K), C10.2, C11.2, C12.2, C13.2, C14.2, C15.2, C16.2, C8.2, C9.2
- net VDD_SPI: now also C15.1
- net at D1.2 (A): now also R13.1
- net GPIO4: now reaches U1.10 (MTMS/GPIO4/FSPIHD/ADC1_CH4)
- net GPIO4: now also J1.8 (Pin_8)
- net GPIO5: now reaches U1.11 (MTDI/GPIO5/FSPIWP/ADC1_CH5)
- net GPIO5: now also J1.7 (Pin_7)
- net GPIO6: now reaches U1.12 (MTCK/GPIO6/FSPICLK/ADC1_CH6)
- net GPIO6: now also J1.6 (Pin_6)
- net GPIO7: now reaches U1.13 (MTDO/GPIO7/FSPID)
- net GPIO7: now also J1.5 (Pin_5)
- net GPIO10: now reaches U1.16 (GPIO10)
- net GPIO10: now also J1.3 (Pin_3)
- net GPIO11: now reaches U1.17 (GPIO11)
- net GPIO11: now also J1.4 (Pin_4)
- net GPIO16: now reaches U1.29 (U0TXD/GPIO16/FSPICS0)
- net GPIO16: now also J1.1 (Pin_1)
- net GPIO17: now reaches U1.30 (U0RXD/GPIO17/FSPICS1)
- net GPIO17: now also J1.2 (Pin_2)
- net GPIO2: now reaches U1.8 (GPIO2/FSPIQ/ADC1_CH2)
- net GPIO2: now also J1.10 (Pin_10)
- net GPIO3: now reaches U1.9 (GPIO3/ADC1_CH3)
- net GPIO3: now also J1.9 (Pin_9)
Other:
- note added: "Connector"
- note added: "Crystal Oscillators"
- note added: "Decoupling capacitors"
- note added: "MCU"
- note added: "Power LED"
- note removed: "Crystals"
- moved on the sheet: AE1, C1, C6, C7, D1, J4, L1, R1, R2, R4, R5, R6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

Commit message: pcb done :yay:
Parts:
- removed AE1: Antenna_Shield, Connector_Coaxial:U.FL_Hirose_U.FL-R-SMT-1_Vertical, symbol Device:Antenna_Shield
- removed J1: Conn_01x10_Pin, symbol Connector:Conn_01x10_Pin
- removed Y2: C252396, symbol Device:Crystal_GND24
- added AE1: Antenna, RF_Antenna:Johanson_2450AT18x100_2400-2500Mhz, symbol Device:Antenna
- added J1: Conn_01x13_Pin, Connector_PinHeader_2.54mm:PinHeader_1x13_P2.54mm_Vertical, symbol Connector:Conn_01x13_Pin
- added JP1: Jumper_2_Bridged, Jumper:SolderJumper-2_P1.3mm_Open_RoundedPad1.0x1.5mm, symbol Jumper:Jumper_2_Bridged
- added L2: 3.3nH, Inductor_SMD:L_0402_1005Metric, symbol Device:L_Small
- added L3: 2.7nH, Inductor_SMD:L_0402_1005Metric, symbol Device:L_Small
- added Y3: Crystal, Crystal:Crystal_SMD_2012-2Pin_2.0x1.2mm, symbol Device:Crystal
- C1, C10, C11, C12, C15, C16, C2, C3, C4, C5, C8, C9: footprint (none) -> Capacitor_SMD:C_0402_1005Metric
- C13: value 470uF -> 1.2pF; footprint (none) -> Capacitor_SMD:C_0402_1005Metric
- C14: footprint (none) -> Capacitor_Tantalum_SMD:CP_EIA-3216-18_Kemet-A
- C6: footprint (none) -> Capacitor_SMD:C_0805_2012Metric
- C7: footprint (none) -> Capacitor_SMD:C_1206_3216Metric
- D1: footprint (none) -> LED_SMD:LED_0805_2012Metric
- J3: footprint (none) -> Connector_Card:microSD_HC_Wuerth_693072010801
- J4: footprint (none) -> Connector_USB:USB_C_Receptacle_HRO_TYPE-C-31-M-12
- L1: footprint (none) -> Inductor_SMD:L_0603_1608Metric
- R1, R10, R11, R12, R13, R2, R3, R4, R5, R6, R7, R8, R9: footprint (none) -> Resistor_SMD:R_0402_1005Metric
- SW1, SW2: footprint (none) -> Button_Switch_SMD:SW_SPST_PTS647_Sx38
- Y1: footprint (none) -> Crystal:Crystal_SMD_3225-4Pin_3.2x2.5mm
Connections:
- net +3.3V: now also J1.3 (Pin_3), JP1.2 (B); no longer C13.1, R13.2
- net +5V: now also J1.2 (Pin_2)
- net ANT: now also C13.1
- net GND: now also J1.1 (Pin_1), L3.1; no longer C13.2
- net GPIO10: now also J1.6 (Pin_6)
- net GPIO11: now also J1.7 (Pin_7)
- net GPIO16: now also J1.4 (Pin_4)
- net GPIO17: now also J1.5 (Pin_5)
- net GPIO2: now also J1.13 (Pin_13)
- net GPIO3: now also J1.12 (Pin_12)
- net GPIO4: now also J1.11 (Pin_11)
- net GPIO5: now also J1.10 (Pin_10)
- net GPIO6: now also J1.9 (Pin_9)
- net GPIO7: now also J1.8 (Pin_8)
- net XTAL_32k_N: now also Y3.1
- net XTAL_32k_P: now also Y3.2
- new net: C13.2, L2.2, L3.2
- new net: AE1.1 (A), L2.1
- new net: JP1.1 (A), R13.2
Other:
- note added: "Antenna"
- title: (none) -> C6dev
- moved on the sheet: C14, D1, R13

Commit message: polishing
Parts:
- L1: value 2uH -> 2.2uH
Changed lines of the file:
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@@
 		(title "C6dev")
 		(date "2025-07-26")
-		(rev "1")
+		(rev "3")
 	)
 	(rectangle
@@
 			)
 		)
-		(property "Value" "2uH"
+		(property "Value" "2.2uH"
 			(at 132.08 138.43 90)
 			(effects

Commit message: silkscreeeen
Connections:
- net GPIO10: now also J1.7 (Pin_7); no longer J1.6 (Pin_6)
- net GPIO11: now also J1.6 (Pin_6); no longer J1.7 (Pin_7)
Changed lines of the file:
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@@
 	)
 	(label "GPIO10"
-		(at 261.62 101.6 180)
+		(at 261.62 104.14 180)
 		(effects
 			(font
@@
 	)
 	(label "GPIO11"
-		(at 261.62 104.14 180)
+		(at 261.62 101.6 180)
 		(effects
 			(font

Commit message: finishing up
Connections:
- net GPIO16: now also J1.5 (Pin_5); no longer J1.4 (Pin_4)
- net GPIO17: now also J1.4 (Pin_4); no longer J1.5 (Pin_5)
Changed lines of the file:
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@@
 	)
 	(label "GPIO16"
-		(at 261.62 96.52 180)
+		(at 261.62 99.06 180)
 		(effects
 			(font
@@
 	)
 	(label "GPIO17"
-		(at 261.62 99.06 180)
+		(at 261.62 96.52 180)
 		(effects
 			(font
